File: Eagle/MICHAv2.0.brd (EAGLE design)
At the start: 110.5 x 83.1 mm, 70 parts, among them IC1 LM4041A12LP, K1 PIN20X2, T1 BSS84, U1 ARDUINO_MKR_ZERO, U2 MIKROE_CLICK_UPGRADE, U3 MAX4528CSA, X1 SS-7188S-A-NF_V2, X2 SS-7188S-A-NF_V2, X3 SS-7188S-A-NF_V2, X4 SS-7188S-A-NF_V2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

Commit message: MAX4528CSA footprint updated
Connections:
- net +5V: now also K1.4
Routing:
- net +5V: track 132.9 -> 135.5 mm
Changed lines of the file:
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@@
 <wire x1="7.94875" y1="-12.05375" x2="5.55625" y2="-12.05375" width="0.4064" layer="16"/>
 <wire x1="17.7373" y1="-2.2652" x2="7.94875" y2="-12.05375" width="0.4064" layer="16"/>
-<contactref element="U3" pad="8"/>
 <contactref element="C15" pad="1"/>
-<wire x1="15.81" y1="31.115" x2="19.18" y2="31.115" width="0.4064" layer="1"/>
-<wire x1="19.18" y1="31.115" x2="19.3675" y2="30.9275" width="0.4064" layer="1"/>
-<wire x1="15.81" y1="31.115" x2="15.81" y2="33.085" width="0.4064" layer="1"/>
-<wire x1="15.81" y1="33.085" x2="15.5575" y2="33.3375" width="0.4064" layer="1"/>
+<wire x1="15.5575" y1="33.3375" x2="15.81" y2="33.085" width="0.4064" layer="1"/>
 <via x="15.5575" y="33.3375" extent="1-16" drill="0.35"/>
 <wire x1="15.5575" y1="33.3375" x2="10.795" y2="38.1" width="0.4064" layer="16"/>
@@
 <wire x1="2.8575" y1="42.545" x2="2.88625" y2="42.57375" width="0.1524" layer="1"/>
 <wire x1="2.88625" y1="42.57375" x2="6.0325" y2="42.57375" width="0.1524" layer="1"/>
+<contactref element="K1" pad="4"/>
+<wire x1="8.22" y1="53.74" x2="10.76" y2="53.74" width="0.4064" layer="1"/>
+<contactref element="U3" pad="8"/>
+<wire x1="15.81" y1="33.085" x2="15.81" y2="31.115" width="0.4064" layer="1"/>
+<wire x1="15.81" y1="31.115" x2="19.18" y2="31.115" width="0.4064" layer="1"/>
+<wire x1="19.18" y1="31.115" x2="19.3675" y2="30.9275" width="0.4064" layer="1"/>
 </signal>
 <signal name="PUMP_PAUSE_BTN">
@@
 <signal name="R_SWITCH">
 <contactref element="K1" pad="36"/>
-<contactref element="U3" pad="4"/>
-<wire x1="13.0175" y1="28.54080625" x2="11.78169375" y2="27.305" width="0.1524" layer="1"/>
-<wire x1="10.86" y1="27.305" x2="11.78169375" y2="27.305" width="0.1524" layer="1"/>
-<wire x1="13.0175" y1="28.54080625" x2="13.0175" y2="36.5125" width="0.1524" layer="1"/>
+<wire x1="13.0175" y1="36.5125" x2="13.0175" y2="28.54080625" width="0.1524" layer="1"/>
 <wire x1="13.0175" y1="36.5125" x2="18.57375" y2="42.06875" width="0.1524" layer="1"/>
 <wire x1="18.57375" y1="42.06875" x2="18.57375" y2="45.72" width="0.1524" layer="1"/>
@@
 <wire x1="30.2807" y1="52.1882" x2="34.0907" y2="52.1882" width="0.1524" layer="1"/>
 <wire x1="36.42621875" y1="55.40375" x2="49.73625" y2="55.40375" width="0.1524" layer="16"/>
+<contactref element="U3" pad="4"/>
+<wire x1="13.0175" y1="28.54080625" x2="11.78169375" y2="27.305" width="0.1524" layer="1"/>
+<wire x1="11.78169375" y1="27.305" x2="10.86" y2="27.305" width="0.1524" layer="1"/>
 </signal>
 <signal name="N$1">
-<contactref element="U3" pad="2"/>
 <wire x1="8.5725" y1="28.73375" x2="8.5725" y2="13.657259375" width="0.1524" layer="1"/>
 <wire x1="8.5725" y1="28.73375" x2="9.68375" y2="29.845" width="0.1524" layer="1"/>
-<wire x1="9.68375" y1="29.845" x2="10.86" y2="29.845" width="0.1524" layer="1"/>
 <contactref element="U2" pad="B"/>
 <wire x1="8.5725" y1="13.657259375" x2="4.813309375" y2="9.81806875" width="0.1524" layer="1"/>
+<contactref element="U3" pad="2"/>
+<wire x1="9.68375" y1="29.845" x2="10.86" y2="29.845" width="0.1524" layer="1"/>
 </signal>
 <signal name="N$10">
-<contactref element="U3" pad="1"/>
-<wire x1="7.9375" y1="28.8925" x2="7.9375" y2="15.875" width="0.1524" layer="1"/>
-<wire x1="7.9375" y1="28.8925" x2="10.16" y2="31.115" width="0.1524" layer="1"/>
-<wire x1="10.16" y1="31.115" x2="10.86" y2="31.115" width="0.1524" layer="1"/>
+<wire x1="7.9375" y1="15.875" x2="7.9375" y2="28.8925" width="0.1524" layer="1"/>
 <contactref element="U2" pad="A"/>
 <wire x1="7.9375" y1="15.875" x2="6.985" y2="14.9225" width="0.1524" layer="1"/>
 <wire x1="6.985" y1="14.9225" x2="4.813309375" y2="14.89806875" width="0.1524" layer="1"/>
+<contactref element="U3" pad="1"/>
+<wire x1="7.9375" y1="28.8925" x2="10.16" y2="31.115" width="0.1524" layer="1"/>
+<wire x1="10.16" y1="31.115" x2="10.86" y2="31.115" width="0.1524" layer="1"/>
 </signal>
 <signal name="R_X">
-<contactref element="U3" pad="7"/>
-<wire x1="15.81" y1="29.845" x2="14.605" y2="29.845" width="0.1524" layer="1"/>
-<wire x1="14.605" y1="29.845" x2="13.97" y2="29.21" width="0.1524" layer="1"/>
+<wire x1="13.97" y1="29.21" x2="14.605" y2="29.845" width="0.1524" layer="1"/>
 <wire x1="13.97" y1="29.21" x2="13.97" y2="17.145" width="0.1524" layer="1"/>
 <wire x1="13.97" y1="17.145" x2="7.9375" y2="11.1125" width="0.1524" layer="1"/>
@@
 <wire x1="9.0297" y1="-2.2225" x2="7.9375" y2="-1.1303" width="0.1524" layer="1"/>
 <wire x1="7.9375" y1="-1.1303" x2="7.9375" y2="-0.9525" width="0.1524" layer="1"/>
+<contactref element="U3" pad="7"/>
+<wire x1="14.605" y1="29.845" x2="15.81" y2="29.845" width="0.1524" layer="1"/>
 </signal>
 <signal name="R_Y">
-<contactref element="U3" pad="6"/>
-<wire x1="15.81" y1="28.575" x2="14.605" y2="28.575" width="0.1524" layer="1"/>
-<wire x1="14.605" y1="28.575" x2="14.2875" y2="28.2575" width="0.1524" layer="1"/>
+<wire x1="14.2875" y1="28.2575" x2="14.605" y2="28.575" width="0.1524" layer="1"/>
 <wire x1="8.255" y1="6.8453" x2="8.255" y2="11.0023375" width="0.1524" layer="1"/>
 <wire x1="14.2875" y1="28.2575" x2="14.2875" y2="17.0348375" width="0.1524" layer="1"/>
@@
 <wire x1="8.5725" y1="3.6445" x2="8.5983" y2="3.6703" width="0.1524" layer="1"/>
 <wire x1="8.5983" y1="3.6703" x2="11.43" y2="3.6703" width="0.1524" layer="1"/>
+<contactref element="U3" pad="6"/>
+<wire x1="14.605" y1="28.575" x2="15.81" y2="28.575" width="0.1524" layer="1"/>
 </signal>
 <signal name="N$11">
